File: component-detector/component-detector.kicad_sch (KiCad schematic)
At the start: 0 parts

Commit message: .
Parts:
- added C1: 0.33uF, symbol Device:C
- added C2: 0.1uF, symbol Device:C
- added C3: 0.1uF, Package_TO_SOT_THT:TO-92_Inline, symbol Device:C
- added Q2: PN2222A, Package_TO_SOT_THT:TO-92_Inline, symbol Transistor_BJT:PN2222A
- added R1: 1k, Package_TO_SOT_SMD:SOT-223-3_TabPin2, symbol Device:R
- added R2: 2k, Package_TO_SOT_SMD:SOT-223-3_TabPin2, symbol Device:R
- added U1: 4N35, Package_DIP:DIP-6_W7.62mm, symbol Isolator:4N35
- added U2: L7805, Package_TO_SOT_THT:TO-220-3_Vertical, symbol Regulator_Linear:L7805
Connections:
- new net: Q2.2 (B), R1.2, R2.1
- new net +12V: C1.2, U2.1 (IN)
- new net +2V5: C3.1, Q2.1 (E)
- new net +5V: C2.2, Q2.3 (C), R1.1, U2.3 (OUT)
- new net GND: C1.1, C2.1, C3.2, R2.2, U2.2 (GND)
Other:
- title: (none) -> Component detector
